Commit message: added function to get a vector of contacts points and corresponding forces in sai2 simulation

File: examples/03-sim_graphics_contact_info/pbot.urdf (robot description, URDF)
Before this commit: robot PBot, 2 links, 1 joints
Links:
- link base_link: geometry 
- link link0: geometry collision box size=0.2 0.2 0.2; visual box size=0.2 0.2 0.2
Joints:
- joint j0: origin xyz=0.000000 0.000000 2.000000 rpy=-0.000000 0.000000 -0.000000 -> xyz=0.000000 0.000000 1.000000 rpy=-0.000000 0.000000 -0.000000
